File: Hardware/Absolute Encoder.kicad_pcb (KiCad board)
At the start: 2 copper layers, 69 x 30 mm, 21 parts, among them J1 PISO_OUT, J2 PISO_IN, U1 74LS165

Commit message: Update Readme
Other:
- board text added: "Absolute Encoder Board"
- board text added: "v1.0"
- board text removed: "PAC18R Encoder Board"
- board text removed: "PISO"
Changed lines of the file:
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@@
 	(gr_poly
 		(pts
-			(xy 227.5 84.5) (xy 232 85.1) (xy 231.3 84.3) (xy 232 83.7) (xy 226.8 84.4)
+			(xy 227.5 84.5) (xy 232 85.2) (xy 231.3 84.3) (xy 232 83.4) (xy 226.8 84.4)
 		)
 		(stroke
@@
 	(gr_poly
 		(pts
-			(xy 177.2 84.7) (xy 181.7 85.3) (xy 181 84.5) (xy 181.7 83.9) (xy 176.5 84.6)
+			(xy 177.2 84.7) (xy 181.7 85.4) (xy 181 84.5) (xy 181.8 83.8) (xy 176.5 84.6)
 		)
 		(stroke
@@
 		)
 	)
-	(gr_text "PISO"
+	(gr_text "v1.0"
 		(at 201.9 77.1 0)
 		(layer "F.SilkS")
@@
 		)
 	)
-	(gr_text "PAC18R Encoder Board"
-		(at 178.2 89.6 0)
+	(gr_text "Absolute Encoder Board"
+		(at 181.4 89.2 0)
 		(layer "F.SilkS")
 		(effects
 			(font
-				(size 2.5 3)
+				(size 2.5 2.5)
 				(thickness 0.3)
 			)
